File: electronics/clock/clock.kicad_sch (KiCad schematic)
At the start: 51 parts, among them J1 Conn_02x03_Counter_Clockwise, J2 Conn_01x02_Male, Q1 2SC1815, Q2 2SC1815, Q3 2SC1815, Q4 2SC1815, Q5 2SC1815, SW2 SW_Push, SW3 SW_Push, SW4 SW_Push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

Commit message: [update] v0.0.1を作成
Parts:
- removed J2: Conn_01x02_Male, Connector_PinSocket_2.54mm:PinSocket_1x02_P2.54mm_Vertical, symbol Connector:Conn_01x02_Male
- added C4, C5: 0.1u, Capacitor_THT:C_Disc_D3.0mm_W1.6mm_P2.50mm, symbol Device:C
- added J2: Barrel_Jack_Switch, Connector_BarrelJack:BarrelJack_Horizontal, symbol Connector:Barrel_Jack_Switch
- J1: footprint Connector_IDC:IDC-Header_2x03_P2.54mm_Horizontal -> Connector_PinHeader_2.54mm:PinHeader_2x03_P2.54mm_Vertical
- R1, R2, R3, R4, R5, R6, R7, R8: value 220 -> 330
- R10, R11, R12, R26, R9: value 47k -> 10k
- R13, R14, R15, R16, R27: value 2.2k -> 3.9k
- R17, R18, R19, R20, R21, R22, R23, R24, R25: value R -> 1k
- Y1: value Crystal -> 16 MHz
Connections:
- net GND: now also C4.2, C5.2, J2.2, J2.3
- net +3V0 renamed +5V
- net +5V: now also C4.1, C5.1, J2.1
- net 7seg-rclk renamed 7SEG_RCLK
- net 7seg-ser renamed 7SEG_SER
- net 7seg-srclk renamed 7SEG_SRCLK
- net dig-1 renamed DIG_1
- net dig-2 renamed DIG_2
- net dig-3 renamed DIG_3
- net dig-4 renamed DIG_4
- net dig-dot renamed DIG_DOT
- net isp-clk renamed ISP_CLK
- net isp-miso renamed ISP_MISO
- net isp-mosi renamed ISP_MOSI
- net isp-reset renamed ISP_RESET
- net sw-clk renamed SW_CLK
- net sw-out renamed SW_OUT
- net sw-s/l renamed SW_S/L
Other:
- title: 4dig-7seg clock -> 4Digit 7Segment Clock
- moved on the sheet: C2, C3, LS1, R1, R17, R18, R19, R2, R20, R21, R22, R23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
